Commit message: Updated HDPR URDF model for 3D Odometry
Signed-off-by: Moritz Schilling <moritz.schilling@dfki.de>

File: data/odometry/hdpr_odometry_model_complete.urdf (robot description, URDF)
Before this commit: robot HDPR, 56 links, 55 joints
Links:
- removed link body_base
- removed link fl_hinge
- removed link fr_hinge
- removed link ml_hinge
- removed link mr_hinge
- removed link rear_bogie
- removed link rl_hinge
- removed link rr_hinge
- added link body; visual box size=1.0 0.7 0.1
- added link camera_assembly; visual mesh filename=./meshes/exoter/bb2_and_tof_camera.stl scale=1 1 1
- added link differential; visual box size=0.7 0.02 0.02
- added link left_rocker; visual box size=0.456 0.02 0.02; visual box size=0.794 0.02 0.02
- added link mast_assembly; visual mesh filename=./meshes/exoter/mast_assembly.stl scale=1 1 1
- added link pan_drive; visual mesh filename=./meshes/exoter/pan_drive.stl scale=1 1 1
- added link right_rocker; visual box size=0.456 0.02 0.02; visual box size=0.794 0.02 0.02
- added link tilt_drive; visual mesh filename=./meshes/exoter/tilt_drive.stl scale=1 1 1
- link fl_fork: geometry visual mesh filename=./meshes/exoter/fork_left.stl scale=1 1 1
- link fl_motor: geometry visual mesh filename=./meshes/exoter/motor_block_fl.stl scale=1 1 1
- link fl_wheel: geometry visual mesh filename=./meshes/exoter/wheel.stl scale=1 1 1
- link fr_fork: geometry visual mesh filename=./meshes/exoter/fork_right.stl scale=1 1 1
- link fr_motor: geometry visual mesh filename=./meshes/exoter/motor_block_rl.stl scale=1 1 1
- link fr_wheel: geometry visual mesh filename=./meshes/exoter/wheel.stl scale=1 1 1
- link left_bogie: geometry visual box size=0.750 0.02 0.02
- link ml_motor: geometry visual mesh filename=./meshes/exoter/motor_middle_left.stl scale=1 1 1
- link ml_wheel: geometry visual mesh filename=./meshes/exoter/wheel.stl scale=1 1 1
- link mr_motor: geometry visual mesh filename=./meshes/exoter/motor_middle_right.stl scale=1 1 1
- link mr_wheel: geometry visual mesh filename=./meshes/exoter/wheel.stl scale=1 1 1
- link right_bogie: geometry visual box size=0.750 0.02 0.02
- link rl_fork: geometry visual mesh filename=./meshes/exoter/fork_left.stl scale=1 1 1
- link rl_motor: geometry visual mesh filename=./meshes/exoter/motor_block_rl.stl scale=1 1 1
- link rl_wheel: geometry visual mesh filename=./meshes/exoter/wheel.stl scale=1 1 1
- link rr_fork: geometry visual mesh filename=./meshes/exoter/fork_right.stl scale=1 1 1
- link rr_motor: geometry visual mesh filename=./meshes/exoter/motor_block_rr.stl scale=1 1 1
- link rr_wheel: geometry visual mesh filename=./meshes/exoter/wheel.stl scale=1 1 1
Joints:
- removed joint fl_mimic
- removed joint fl_walking
- removed joint fr_mimic
- removed joint fr_walking
- removed joint ml_mimic
- removed joint ml_walking
- removed joint mr_mimic
- removed joint mr_walking
- removed joint rear_passive
- removed joint rl_mimic
- removed joint rl_walking
- removed joint rr_mimic
- removed joint rr_walking
- added joint front_passive: type continuous, parent body, child differential, origin xyz=0.5 0 0 rpy=0.0 0.0 0.00, axis 1 0 0 , limit lower=-1.6 upper=1.6 effort=100 velocity=6.28
- added joint left_bogie_to_ml_motor: type fixed, parent left_bogie, child ml_motor, origin xyz=0.375 0 0 rpy=0 0.0 0, axis 0 1 0
- added joint left_bogie_to_rl_motor: type fixed, parent left_bogie, child rl_motor, origin xyz=-0.375 0 0 rpy=0 0.0 0, axis 0 1 0
- added joint left_rocker_bogie: type continuous, parent left_rocker, child left_bogie, origin xyz=-0.375 0.0 -0.260 rpy=0 0.0 0, axis 0 1 0, limit lower=-0.17 upper=1.6 effort=100 velocity=6.28
- added joint left_rocker_to_motor: type fixed, parent left_rocker, child fl_motor, origin xyz=0.750 0 -0.260 rpy=0 0.0 0, axis 0 1 0
- added joint mast_joint: type fixed, parent body, child mast_assembly, origin xyz=0.076 0.0 0.0 rpy=0 0.0 0, limit lower=-1.6 upper=1.6 effort=100 velocity=6.28
- added joint mast_top_joint: type fixed, parent mast_assembly, child pan_drive, origin xyz=0.0 0.0 0.64 rpy=0 0.0 0, limit lower=-1.6 upper=1.6 effort=100 velocity=6.28
- added joint pan_joint: type continuous, parent pan_drive, child tilt_drive, origin xyz=0.0 0.0 0.0 rpy=0 0.0 0, axis 0 0 1, limit lower=-1.6 upper=1.6 effort=100 velocity=6.28
- added joint right_bogie_to_ml_motor: type fixed, parent right_bogie, child mr_motor, origin xyz=0.375 0 0 rpy=0 0.0 0, axis 0 1 0
- added joint right_bogie_to_rl_motor: type fixed, parent right_bogie, child rr_motor, origin xyz=-0.375 0 0 rpy=0 0.0 0, axis 0 1 0
- added joint right_rocker_bogie: type continuous, parent right_rocker, child right_bogie, origin xyz=-0.375 0 -0.260 rpy=0 0.0 0, axis 0 1 0, limit lower=-0.17 upper=1.6 effort=100 velocity=6.28
- added joint right_rocker_to_motor: type fixed, parent right_rocker, child fr_motor, origin xyz=0.750 0 -0.260 rpy=0 0.0 0, axis 0 1 0
- added joint tilt_joint: type continuous, parent tilt_drive, child camera_assembly, origin xyz=0.0 0.0 0.03 rpy=0 0.0 0, axis 0 1 0, limit lower=-1.6 upper=1.6 effort=100 velocity=6.28
- joint fl_contact: origin xyz=0 0.0 -0.072703 rpy=0 0.00 0 -> xyz=0 0.0 -0.125 rpy=0 0.00 0; type fixed -> continuous
- joint fl_drive: limit lower=-3.14 upper=3.14 effort=100 velocity=60.28 -> lower=-3.14 upper=3.14 effort=100 velocity=6.28
- joint fl_slipx: type fixed -> prismatic
- joint fl_slipy: type fixed -> prismatic
- joint fl_slipz: type fixed -> continuous
- joint fl_translation: type fixed -> prismatic
- joint fr_contact: origin xyz=0 0.0 -0.072703 rpy=0 0.00 0 -> xyz=0 0.0 -0.125 rpy=0 0.00 0; type fixed -> continuous
- joint fr_drive: limit lower=-3.14 upper=3.14 effort=100 velocity=60.28 -> lower=-3.14 upper=3.14 effort=100 velocity=6.28
- joint fr_slipx: type fixed -> prismatic
- joint fr_slipy: type fixed -> prismatic
- joint fr_slipz: type fixed -> continuous
- joint fr_translation: type fixed -> prismatic
- joint left_passive: child left_bogie -> left_rocker; origin xyz=0.1325 0.223 0 rpy=0 0.00 0 -> xyz=0.0 0.41 0 rpy=0 0.00 0; parent body_base -> body; type fixed -> continuous
- joint ml_contact: origin xyz=0 0.0 -0.072703 rpy=0 0.00 0 -> xyz=0 0.0 -0.125 rpy=0 0.00 0; type fixed -> continuous
- joint ml_drive: limit lower=-3.14 upper=3.14 effort=100 velocity=60.28 -> lower=-3.14 upper=3.14 effort=100 velocity=6.28
- joint ml_slipx: type fixed -> prismatic
- joint ml_slipy: type fixed -> prismatic
- joint ml_slipz: type fixed -> continuous
- joint ml_translation: type fixed -> prismatic
- joint mr_contact: origin xyz=0 0.0 -0.072703 rpy=0 0.00 0 -> xyz=0 0.0 -0.125 rpy=0 0.00 0; type fixed -> continuous
- joint mr_drive: limit lower=-3.14 upper=3.14 effort=100 velocity=60.28 -> lower=-3.14 upper=3.14 effort=100 velocity=6.28
- joint mr_slipx: type fixed -> prismatic
- joint mr_slipy: type fixed -> prismatic
- joint mr_slipz: type fixed -> continuous
- joint mr_translation: type fixed -> prismatic
- joint right_passive: child right_bogie -> right_rocker; mimic (none) -> joint=left_passive multiplier=-1 offset=0; origin xyz=0.1325 -0.223 0 rpy=0 0.00 0 -> xyz=0.0 -0.41 0.0 rpy=0 0.00 0; parent body_base -> body; type fixed -> continuous
- joint rl_contact: origin xyz=0 0.0 -0.072703 rpy=0 0.00 0 -> xyz=0 0.0 -0.125 rpy=0 0.00 0; type fixed -> continuous
- joint rl_drive: limit lower=-3.14 upper=3.14 effort=100 velocity=60.28 -> lower=-3.14 upper=3.14 effort=100 velocity=6.28
- joint rl_slipx: type fixed -> prismatic
- joint rl_slipy: type fixed -> prismatic
- joint rl_slipz: type fixed -> continuous
- joint rl_translation: type fixed -> prismatic
- joint rr_contact: origin xyz=0 0.0 -0.072703 rpy=0 0.00 0 -> xyz=0 0.0 -0.125 rpy=0 0.00 0; type fixed -> continuous
- joint rr_drive: limit lower=-3.14 upper=3.14 effort=100 velocity=60.28 -> lower=-3.14 upper=3.14 effort=100 velocity=6.28
- joint rr_slipx: type fixed -> prismatic
- joint rr_slipy: type fixed -> prismatic
- joint rr_slipz: type fixed -> continuous
- joint rr_translation: type fixed -> prismatic

Commit message: Removed unnecessary joints and temporarily fixed the ones we don't know about in HDPR
Signed-off-by: Moritz Schilling <moritz.schilling@dfki.de>

File: data/odometry/hdpr_odometry_model_complete.urdf (robot description, URDF)
Before this commit: robot HDPR, 56 links, 55 joints
Links:
- removed link camera_assembly
- removed link differential
- removed link mast_assembly
- removed link pan_drive
- removed link tilt_drive
Joints:
- removed joint front_passive
- removed joint mast_joint
- removed joint mast_top_joint
- removed joint pan_joint
- removed joint tilt_joint
- joint left_passive: type continuous -> fixed
- joint left_rocker_bogie: type continuous -> fixed
- joint right_passive: type continuous -> fixed
- joint right_rocker_bogie: type continuous -> fixed

Commit message: Made changes to config files so that Threed Odometry works for HDPR

File: data/odometry/hdpr_odometry_model_complete.urdf (robot description, URDF)
Before this commit: robot HDPR, 51 links, 50 joints
Joints:
- joint left_passive: type fixed -> continuous
- joint left_rocker_bogie: type fixed -> continuous
- joint right_passive: type fixed -> continuous
- joint right_rocker_bogie: type fixed -> continuous
